Commit message: Matching the frames between kinematic model, urdf and motion capture system

File: omni_description/robots/omnipointer.urdf (robot description, URDF)
Before this commit: robot omnipointer, 16 links, 15 joints
Joints:
- joint arm_joint_0: origin xyz=-0.021 0 0 rpy=0 0 0 -> xyz=0.021 0 0 rpy=0 0 0
- joint plate_joint: origin xyz=0.148 0 0.061 rpy=0 0 0 -> xyz=-0.148 0 0.061 rpy=0 0 0

File: omni_description/robots/omnipointer.urdf.xacro (robot description, xacro)
@@ -23,8 +23,8 @@
   <xacro:youbot_base name="base"/>
   <xacro:omni_plate name="plate" parent="base_link">
-    <origin xyz="0.148 0 0.061" rpy="0 0 0" />
+    <origin xyz="-0.148 0 0.061" rpy="0 0 0" />
   </xacro:omni_plate>
   <xacro:omnipointer_arm name="arm" parent="plate_link">
-    <origin xyz="-0.021 0 0" rpy="0 0 0" />
+    <origin xyz="0.021 0 0" rpy="0 0 0" />
   </xacro:omnipointer_arm>
 </robot>

Commit message: Still matching the frames between kinematic model, urdf and motion capture system

File: omni_description/robots/omnipointer.urdf (robot description, URDF)
Before this commit: robot omnipointer, 16 links, 15 joints
Joints:
- joint arm_joint_0: origin xyz=0.021 0 0 rpy=0 0 0 -> xyz=0.021 0 0 rpy=0 0 3.14159265359

File: omni_description/robots/omnipointer.urdf.xacro (robot description, xacro)
@@ -26,5 +26,5 @@
   </xacro:omni_plate>
   <xacro:omnipointer_arm name="arm" parent="plate_link">
-    <origin xyz="0.021 0 0" rpy="0 0 0" />
+    <origin xyz="0.021 0 0" rpy="0 0 ${M_PI}" />
   </xacro:omnipointer_arm>
 </robot>
