Commit message: Integration of the arm in the full robot

File: omni_description/robots/omnigrasper.urdf.xacro (robot description, xacro)
@@ -21,8 +21,10 @@
        the origin block defines where the component is w.r.t its parent (in this case the parent
        is the world frame). For more, see http://www.ros.org/wiki/xacro -->
-  <!-- <xacro:youbot_base name="base"/> -->
-  <!-- <xacro:omni_plate name="plate" parent="base_link">
+  <xacro:youbot_base name="base"/>
+  <xacro:omni_plate name="plate" parent="base_link">
     <origin xyz="-0.148 0 0.061" rpy="0 0 0" />
-  </xacro:omni_plate> -->
-  <xacro:omnigrasper_arm/>
+  </xacro:omni_plate>
+  <xacro:omnigrasper_arm name="arm" parent="plate_link">
+    <origin xyz="0 0 0.004" rpy="0 0 0" />
+  </xacro:omnigrasper_arm>
 </robot>

File: omni_description/urdf/omnigrasper_arm/arm.urdf.xacro (robot description, xacro)
@@ -2,15 +2,13 @@
 <robot name="omnigrasper" xmlns:xacro="http://ros.org/wiki/xacro">
     <!-- Xacro macro for the arm -->
-    <xacro:macro name="omnigrasper_arm">
-        <link name="plate">
-            <!-- <xacro:visuals_collisions_arm_0/> -->
-            <visual>
-                <geometry>
-                    <box size="0.25 0.25 0.10"/>
-                </geometry>
-            </visual>
-        </link>
-        <joint name="plate_arm_0" type="fixed">
-            <parent link="plate"/>
+    <xacro:macro name="omnigrasper_arm" params="parent name *origin">
+        <joint name="${parent}_${name}_base" type="fixed">
+            <parent link="${parent}"/>
+            <child link="${name}_base"/>
+            <xacro:insert_block name="origin"/>
+        </joint>
+        <link name="${name}_base"/>
+        <joint name="${name}_base_arm_0" type="fixed">
+            <parent link="${name}_base"/>
             <child link="arm_0"/>
             <origin xyz="0 0 0.141"/>
@@ -19,6 +17,7 @@
             <!-- <xacro:visuals_collisions_arm_0/> -->
             <visual>
+                <origin xyz="0 0 ${-0.001*(54/2+6+108/2)}" rpy="0 0 0"/>
                 <geometry>
-                    <box size="0.05 0.05 0.05"/>
+                    <box size="0.054 0.054 0.108"/>
                 </geometry>
             </visual>
@@ -115,8 +114,8 @@
         <joint name="arm_5_end" type="fixed">
             <parent link="arm_5"/>
-            <child link="arm_end"/>
+            <child link="arm_link"/>
             <origin xyz="0 0.039 -0.006"/>
         </joint>
-        <link name="arm_end">
+        <link name="arm_link">
             <!-- <xacro:visuals_collisions_arm_0/> -->
             <!-- <visual>
