Commit message: refactoring of Xacro models

File: omni_description/urdf/omnigrasper_arm/arm.urdf.xacro (robot description, xacro)
@@ -1,9 +1,6 @@
 <?xml version="1.0"?>
 <robot name="omnigrasper" xmlns:xacro="http://ros.org/wiki/xacro">
-    <xacro:include filename="$(find omni_description)/urdf/common.xacro" />
-    <xacro:leg/>
-    <!-- TODO use the box link macro in common.xacro -->
     <!-- Xacro macro for the arm -->
-    <xacro:macro name="leg">
+    <xacro:macro name="omnigrasper_arm">
         <link name="plate">
             <!-- <xacro:visuals_collisions_arm_0/> -->

Commit message: Geometric, Dynamic model finished and limits defined
All frames of the arm are now defined and should be correct. The first approximation for the dynamic model is also done.

Joint limits as well as torque and velocity limits are defined based on measurements on the finished arm and informations from the manufacturer.

File: omni_description/urdf/omnigrasper_arm/arm.urdf.xacro (robot description, xacro)
@@ -27,5 +27,6 @@
             <parent link="arm_0"/>
             <child link="arm_1"/>
-            <!-- <limit effort="${5}" velocity="${5}" lower="${-M_PI}" upper="${M_PI}"/> -->
+            <limit effort="2.5" velocity="${28.7*M_PI/30}"
+                lower="${-M_PI}" upper="${M_PI}"/>
             <origin rpy="0 0 0" xyz="0 0 0"/>
             <axis xyz="0 0 1"/>
@@ -34,31 +35,13 @@
         <link name="arm_1">
             <!-- TODO Parts to add : frame adaptor FRP54-A110K, idler FRP54-I110 -->
-            <xacro:box_vci name="arm_1" mass="0.855"
+            <xacro:box_vci name="H54-200-S500" mass="0.855"
                 size_x="0.054" size_y="0.132" size_z="0.054"
                 xyz="0 0 0"/>
-            <!-- <xacro:property name="arm_1_mass" value="0.855" />
-            <xacro:property name="arm_1_lx" value="0.054" />
-            <xacro:property name="arm_1_ly" value="0.132" />
-            <xacro:property name="arm_1_lz" value="0.054" />
-            <!-- <xacro:visuals_collisions_arm_1/> --
-            <visual> <!-- H54-200-S500 --
-                <geometry>
-                    <box size="${arm_1_lx} ${arm_1_ly} ${arm_1_lz}"/>
-                </geometry>
-            </visual>
-            <inertial> <!-- H54-200-S500 --
-                <!-- center of mass --
-                <origin rpy="0 0 0" xyz="0 0 0"/>
-                <mass value="${arm_1_mass}"/>
-                <!-- box inertia: 1/12*m(y^2+z^2), ... --
-                <inertia ixx="${1/12*arm_1_mass*(arm_1_ly**2 + arm_1_lz**2)}" ixy="0" ixz="0"
-                    iyy="${1/12*arm_1_mass*(arm_1_lx**2 + arm_1_lz**2)}" iyz="0"
-                    izz="${1/12*arm_1_mass*(arm_1_lx**2 + arm_1_ly**2)}"/>
-            </inertial> -->
         </link>
         <joint name="arm_1_2" type="revolute">
             <parent link="arm_1"/>
             <child link="arm_2"/>
-            <!-- <limit effort="${5}" velocity="${5}" lower="${-M_PI}" upper="${M_PI}"/> -->
+            <limit effort="44.7" velocity="${33.1*M_PI/30}"
+                lower="${1.34-M_PI}" upper="${4.94-M_PI}"/>
             <origin rpy="${M_PI/2} ${-M_PI/2} 0" xyz="0 0 0"/>
             <axis xyz="0 0 1"/>
@@ -66,160 +49,81 @@
         </joint>
         <link name="arm_2">
-            <xacro:visuals_collisions_arm_2/>
-            <!-- TODO Parts to add : modified (by us) frame FRP54-H220, modified
-            (by us) frame adaptor FRP54-H120K (modified by us), idler FRP54-I110 -->
             <!-- <xacro:visuals_collisions_arm_2/> -->
+            <!-- TODO Parts to add : modified (by us) frame FRP54-H220, (modified
+            by us) frame adaptor FRP54-A110K (modified by us), idler FRP54-I110 -->
+            <!-- TODO: take the moments of inertia provided by manufacturer -->
             <xacro:box_vci name="profile_2" mass="${1.38*0.180}"
                 size_x="0.180" size_y="0.040" size_z="0.040"
                 xyz="${0.001*(51+180/2)} 0 0"/>
-            <!-- <xacro:property name="profile_2_mass" value="${1.38*0.180}" />
-            <xacro:property name="profile_2_lx" value="0.180" />
-            <xacro:property name="profile_2_ly" value="0.040" />
-            <xacro:property name="profile_2_lz" value="0.040" />
-            <visual> <!-- aluminium profile --> -->
-                <!-- <origin rpy="0 0 0" xyz="${0.001*(51+180/2)} 0 0"/>
-                <geometry name="profile_2">
-                    <box size="${profile_2_lx} ${profile_2_ly} ${profile_2_lz}"/>
-                </geometry>
-            </visual>
-            <inertial> <!-- aluminium profile --> -->
-                <!-- TODO: take the moments of inertia provided by manufacturer -->
-                <!-- center of mass -->
-                <!-- <origin rpy="0 0 0" xyz="${0.001*(51+180/2)} 0 0"/>
-                <mass value="${profile_2_mass}"/> -->
-                <!-- box inertia: 1/12*m(y^2+z^2), ... -->
-                <!-- <inertia ixx="${1/12*profile_2_mass*(profile_2_ly**2 + profile_2_lz**2)}" ixy="0" ixz="0"
-                    iyy="${1/12*profile_2_mass*(profile_2_lx**2 + profile_2_lz**2)}" iyz="0"
-                    izz="${1/12*profile_2_mass*(profile_2_lx**2 + profile_2_ly**2)}"/>
-            </inertial> -->
             <xacro:box_vci name="L54_50_S500" mass="0.662"
                 size_x="0.054" size_y="0.054" size_z="0.114"
-                xyz="${0.001*(51+180/2)} 0 0"/>
-            <!-- <xacro:property name="L54_50_S500_mass" value="0.662" />
-            <xacro:property name="L54_50_S500_lx" value="0.054" />
-            <xacro:property name="L54_50_S500_ly" value="0.054" />
-            <xacro:property name="L54_50_S500_lz" value="0.114" />
-            <visual> <!-- L54-50-S500 --> -->
-                <!-- <origin rpy="0 0 0" xyz="${0.001*(51+180+6+54/2)} 0 0"/>
-                <geometry name="L54_50_S500"> <!-- L54-50-S500 --> -->
-                    <!-- <box size="${L54_50_S500_lx} ${L54_50_S500_ly} ${L54_50_S500_lz}"/>
-                </geometry>
-            </visual>
-            <inertial> <!-- L54-50-S500 --> -->
-                <!-- center of mass -->
-                <!-- <origin rpy="0 0 0" xyz="${0.001*(51+180+6+54/2)} 0 0"/>
-                <mass value="${L54_50_S500_mass}"/> -->
-                <!-- box inertia: 1/12*m(y^2+z^2), ... -->
-                <!-- <inertia ixx="${1/12*L54_50_S500_mass*(L54_50_S500_ly**2 + L54_50_S500_lz**2)}" ixy="0" ixz="0"
-                    iyy="${1/12*L54_50_S500_mass*(L54_50_S500_lx**2 + L54_50_S500_lz**2)}" iyz="0"
-                    izz="${1/12*L54_50_S500_mass*(L54_50_S500_lx**2 + L54_50_S500_ly**2)}"/>
-            </inertial> -->
+                xyz="${0.001*(51+180+6+54/2)} 0 0"/>
         </link>
-        <joint name="arm_0_1" type="revolute">
-            <parent link="arm_0"/>
-            <child link="arm_1"/>
-            <!-- <limit effort="${joint_1_eff}" lower="${-joint_1_lim}" upper="${joint_1_lim}" velocity="${joint_vel}"/> -->
-            <origin rpy="0 0 0" xyz="0 0 0"/>
+        <joint name="arm_2_3" type="revolute">
+            <parent link="arm_2"/>
+            <child link="arm_3"/>
+            <limit effort="14" velocity="${16*M_PI/30}"
+                lower="${1.32-M_PI}" upper="${4.80-M_PI}"/>
+            <origin rpy="0 0 ${-M_PI/2}" xyz="0.264 0 0"/>
             <axis xyz="0 0 1"/>
             <!-- <dynamics damping="${joint_dmp}"/> -->
         </joint>
-        <link name="arm_1">
-            <xacro:visuals_collisions_arm_1/>
-            <inertial>
-                <!-- Parts to add : frame adaptor FRP54-A110K, idler FRP54-I110 -->
-                <xacro:property name="arm_1_mass" value="0.855" />
-                <xacro:property name="arm_1_lx" value="0.054" />
-                <xacro:property name="arm_1_ly" value="0.132" />
-                <xacro:property name="arm_1_lz" value="0.054" />
-                <!-- center of mass -->
-                <origin rpy="0 0 0" xyz="0 0 ${6+54/2}"/>
-                <mass value="arm_1_mass"/>
-                <!-- box inertia: 1/12*m(y^2+z^2), ... -->
-                <inertia ixx="${1/12*arm_1_mass*(arm_1_ly**2 + arm_1_lz**2)}" ixy="0" ixz="0" iyy="${1/12*arm_1_mass*(arm_1_lx**2 + arm_1_lz**2)}" iyz="0" izz="${1/12*arm_1_mass*(arm_1_lx**2 + arm_1_ly**2)}"/>
-            </inertial>
+        <link name="arm_3">
+            <!-- <xacro:visuals_collisions_arm_3/> -->
+            <!-- TODO Parts to add : modified (by us) frame FRP54-H120, modofied
+            (by us) frame adaptor FRP54-A110K, idler FRP54-I110 -->
+            <!-- TODO: take the moments of inertia provided by manufacturer -->
+            <xacro:box_vci name="profile_3" mass="${1.38*0.060}"
+                size_x="0.040" size_y="0.060" size_z="0.040"
+                xyz="0 ${0.001*(51+60/2)} 0"/>
+            <xacro:box_vci name="L54_30_S500" mass="0.612"
+                size_x="0.054" size_y="0.108" size_z="0.054"
+                xyz="0 ${0.001*(51+60+6+108/2)} 0"/>
         </link>
-        <joint name="arm_0_1" type="revolute">
-            <parent link="arm_0"/>
-            <child link="arm_1"/>
-            <!-- <limit effort="${joint_1_eff}" lower="${-joint_1_lim}" upper="${joint_1_lim}" velocity="${joint_vel}"/> -->
-            <origin rpy="0 0 0" xyz="0 0 0"/>
+        <joint name="arm_3_4" type="revolute">
+            <parent link="arm_3"/>
+            <child link="arm_4"/>
+            <limit effort="2.5" velocity="${28.7*M_PI/30}" lower="${-M_PI}" upper="${M_PI}"/>
+            <origin rpy="${-M_PI/2} 0 0" xyz="0 0.252 0"/>
             <axis xyz="0 0 1"/>
             <!-- <dynamics damping="${joint_dmp}"/> -->
         </joint>
-        <link name="arm_1">
-            <xacro:visuals_collisions_arm_1/>
-            <inertial>
-                <!-- Parts to add : frame adaptor FRP54-A110K, idler FRP54-I110 -->
-                <xacro:property name="arm_1_mass" value="0.855" />
-                <xacro:property name="arm_1_lx" value="0.054" />
-                <xacro:property name="arm_1_ly" value="0.132" />
-                <xacro:property name="arm_1_lz" value="0.054" />
-                <!-- center of mass -->
-                <origin rpy="0 0 0" xyz="0 0 ${6+54/2}"/>
-                <mass value="arm_1_mass"/>
-                <!-- box inertia: 1/12*m(y^2+z^2), ... -->
-                <inertia ixx="${1/12*arm_1_mass*(arm_1_ly**2 + arm_1_lz**2)}" ixy="0" ixz="0" iyy="${1/12*arm_1_mass*(arm_1_lx**2 + arm_1_lz**2)}" iyz="0" izz="${1/12*arm_1_mass*(arm_1_lx**2 + arm_1_ly**2)}"/>
-            </inertial>
+        <link name="arm_4">
+            <!-- <xacro:visuals_collisions_arm_4/> -->
+            <!-- TODO Parts to add : modified (by us) frame adaptor FRP54-A110K,
+            idler FRP42-I110 -->
+            <xacro:box_vci name="L42_10_S300" mass="0.257"
+                size_x="0.042" size_y="0.072" size_z="0.042"
+                xyz="0 0 0"/>
         </link>
-        <joint name="leg_${index}_2_3" type="revolute">
-            <parent link="leg_${index}_2"/>
-            <child link="leg_${index}_3"/>
-            <limit effort="${joint_eff}" lower="${-joint_lim}" upper="${joint_lim}" velocity="${joint_vel}"/>
-            <origin rpy="0 0 0" xyz="0 ${arm_1_length} 0"/>
-            <axis xyz="-1 0 0"/>
-            <dynamics damping="${joint_dmp}"/>
+        <joint name="arm_4_5" type="revolute">
+            <parent link="arm_4"/>
+            <child link="arm_5"/>
+            <limit effort="1.2" velocity="${29.7*M_PI/30}" lower="${-M_PI/2}" upper="${M_PI/2}"/>
+            <origin rpy="${M_PI/2} 0 0" xyz="0 0 0"/>
+            <axis xyz="0 0 1"/>
+            <!-- <dynamics damping="${joint_dmp}"/> -->
         </joint>
-        <link name="leg_${index}_3">
-            <xacro:visuals_collisions_leg_3/>
-            <inertial>
-                <!-- CENTER OF MASS -->
-                <origin rpy="${PI_2} 0 0" xyz="0 ${leg3_length/2} 0"/>
-                <mass value="${leg3_mass}"/>
-                <!-- box inertia: 1/12*m(y^2+z^2), ... -->
-                <inertia ixx="${1/12*leg3_mass*(leg3_width*leg3_width+leg3_length*leg3_length)}" ixy="0" ixz="0" iyy="${1/12*leg3_mass*(leg3_width*leg3_width+leg3_length*leg3_length)}" iyz="0" izz="${1/12*leg3_mass*(2*leg3_width*leg3_width)}"/>
-            </inertial>
+        <link name="arm_5">
+            <!-- <xacro:visuals_collisions_arm_5/> -->
+            <!-- TODO Parts to add : frame FRP42-H220 -->
+            <!-- FIXME: The weight is made up, as well as the center of mass -->
+            <xacro:box_vci name="L42_10_S300" mass="0.0857"
+                size_x="0.042" size_y="0.006" size_z="0.082"
+                xyz="0 0.039 -0.006"/>
         </link>
-        <joint name="force_sensor_${index}_fix" type="fixed">
-            <parent link="leg_${index}_3"/>
-            <child link="force_sensor_${index}"/>
-            <origin rpy="${PI} 0 ${PI_2}" xyz="0 ${force_y_offset} -${force_z_offset}"/>
+        <joint name="arm_5_end" type="fixed">
+            <parent link="arm_5"/>
+            <child link="arm_end"/>
+            <origin xyz="0 0.039 -0.006"/>
         </joint>
-        <link name="force_sensor_${index}"/>
-        <!-- Description used by our Dart simulator -->
-        <dart_sensor type="force">
-          <link>force_sensor_${index}</link>
-          <frequency>1000</frequency>
-          <topic>optoforce_${index}</topic>
-        </dart_sensor>
-        <transmission name="tran${index}1">
-            <type>transmission_interface/SimpleTransmission</type>
-            <joint name="body_leg_${index}">
-                <hardwareInterface>PositionJointInterface</hardwareInterface>
-            </joint>
-            <actuator name="motor${index}1">
-                <hardwareInterface>PositionJointInterface</hardwareInterface>
-                <mechanicalReduction>1</mechanicalReduction>
-            </actuator>
-        </transmission>
-        <transmission name="tran${index}2">
-            <type>transmission_interface/SimpleTransmission</type>
-            <joint name="arm_1_2">
-                <hardwareInterface>PositionJointInterface</hardwareInterface>
-            </joint>
-            <actuator name="motor${index}2">
-                <hardwareInterface>PositionJointInterface</hardwareInterface>
-                <mechanicalReduction>1</mechanicalReduction>
-            </actuator>
-        </transmission>
-        <transmission name="tran${index}3">
-            <type>transmission_interface/SimpleTransmission</type>
-            <joint name="leg_${index}_2_3">
-                <hardwareInterface>PositionJointInterface</hardwareInterface>
-            </joint>
-            <actuator name="motor${index}2">
-                <hardwareInterface>PositionJointInterface</hardwareInterface>
-                <mechanicalReduction>1</mechanicalReduction>
-            </actuator>
-        </transmission>
+        <link name="arm_end">
+            <!-- <xacro:visuals_collisions_arm_0/> -->
+            <!-- <visual>
+                <geometry>
+                    <box size="0.0025 0.03 0.0025"/>
+                </geometry>
+            </visual> -->
+        </link>
     </xacro:macro>
     <!-- end of arm links/joints -->

Commit message: cleanup of some old comments

File: omni_description/urdf/omnigrasper_arm/arm.urdf.xacro (robot description, xacro)
@@ -15,5 +15,4 @@
         </joint>
         <link name="arm_0">
-            <!-- <xacro:visuals_collisions_arm_0/> -->
             <visual>
                 <origin xyz="0 0 ${-0.001*(54/2+6+108/2)}" rpy="0 0 0"/>
@@ -31,5 +30,4 @@
             <origin rpy="0 0 0" xyz="0 0 0"/>
             <axis xyz="0 0 1"/>
-            <!-- <dynamics damping="${joint_dmp}"/> -->
         </joint>
         <link name="arm_1">
@@ -46,8 +44,6 @@
             <origin rpy="${M_PI/2} ${-M_PI/2} 0" xyz="0 0 0"/>
             <axis xyz="0 0 1"/>
-            <!-- <dynamics damping="${joint_dmp}"/> -->
         </joint>
         <link name="arm_2">
-            <!-- <xacro:visuals_collisions_arm_2/> -->
             <!-- TODO Parts to add : modified (by us) frame FRP54-H220, (modified
             by us) frame adaptor FRP54-A110K (modified by us), idler FRP54-I110 -->
@@ -67,8 +63,6 @@
             <origin rpy="0 0 ${-M_PI/2}" xyz="0.264 0 0"/>
             <axis xyz="0 0 1"/>
-            <!-- <dynamics damping="${joint_dmp}"/> -->
         </joint>
         <link name="arm_3">
-            <!-- <xacro:visuals_collisions_arm_3/> -->
             <!-- TODO Parts to add : modified (by us) frame FRP54-H120, modofied
             (by us) frame adaptor FRP54-A110K, idler FRP54-I110 -->
@@ -87,8 +81,6 @@
             <origin rpy="${-M_PI/2} 0 0" xyz="0 0.252 0"/>
             <axis xyz="0 0 1"/>
-            <!-- <dynamics damping="${joint_dmp}"/> -->
         </joint>
         <link name="arm_4">
-            <!-- <xacro:visuals_collisions_arm_4/> -->
             <!-- TODO Parts to add : modified (by us) frame adaptor FRP54-A110K,
             idler FRP42-I110 -->
@@ -103,8 +95,6 @@
             <origin rpy="${M_PI/2} 0 0" xyz="0 0 0"/>
             <axis xyz="0 0 1"/>
-            <!-- <dynamics damping="${joint_dmp}"/> -->
         </joint>
         <link name="arm_5">
-            <!-- <xacro:visuals_collisions_arm_5/> -->
             <!-- TODO Parts to add : frame FRP42-H220 -->
             <!-- FIXME: The weight is made up, as well as the center of mass -->
@@ -118,12 +108,5 @@
             <origin xyz="0 0.039 -0.006"/>
         </joint>
-        <link name="arm_link">
-            <!-- <xacro:visuals_collisions_arm_0/> -->
-            <!-- <visual>
-                <geometry>
-                    <box size="0.0025 0.03 0.0025"/>
-                </geometry>
-            </visual> -->
-        </link>
+        <link name="arm_link"/>
     </xacro:macro>
     <!-- end of arm links/joints -->

Commit message: reshape the URDF for Inertias to be accepted by Dart

File: omni_description/urdf/omnigrasper_arm/arm.urdf.xacro (robot description, xacro)
@@ -52,4 +52,11 @@
                 size_x="0.180" size_y="0.040" size_z="0.040"
                 xyz="${0.001*(51+180/2)} 0 0" color="omni/Green"/>
+        </link>
+        <joint name="arm_2_sub" type="fixed">
+            <parent link="arm_2"/>
+            <child link="arm_2_sub"/>
+            <origin xyz="0 0 0"/>
+        </joint>
+        <link name="arm_2_sub">
             <xacro:box_vci name="L54_50_S500" mass="0.662"
                 size_x="0.054" size_y="0.054" size_z="0.114"
@@ -71,4 +78,14 @@
                 size_x="0.040" size_y="0.060" size_z="0.040"
                 xyz="0 ${0.001*(51+60/2)} 0" color="omni/Yellow"/>
+            <xacro:box_vci name="L54_30_S500" mass="0.612"
+                size_x="0.054" size_y="0.108" size_z="0.054"
+                xyz="0 ${0.001*(51+60+6+108/2)} 0" color="omni/Yellow"/>
+        </link>
+        <joint name="arm_3_sub" type="fixed">
+            <parent link="arm_3"/>
+            <child link="arm_3_sub"/>
+            <origin xyz="0 0 0"/>
+        </joint>
+        <link name="arm_3_sub">
             <xacro:box_vci name="L54_30_S500" mass="0.612"
                 size_x="0.054" size_y="0.108" size_z="0.054"

Commit message: Add collision representation of arm base

File: omni_description/urdf/omnigrasper_arm/arm.urdf.xacro (robot description, xacro)
@@ -22,4 +22,10 @@
                 <material name="omni/Blue"/>
             </visual>
+            <collision>
+                <origin xyz="0 0 ${-0.001*(54/2+6+108/2)}" rpy="0 0 0"/>
+                <geometry>
+                    <box size="0.054 0.054 0.108"/>
+                </geometry>
+            </collision>
         </link>
         <joint name="arm_0_1" type="revolute">
