Commit message: testing a refactor

File: omni_description/urdf/common.xacro (robot description, xacro)
@@ -26,3 +26,27 @@
           </link>
     </xacro:macro>
+    <xacro:macro name="box_vci" params="name mass size_x size_y size_z xyz">
+        <!-- For Box Visual Collision Intertial -->
+        <visual>
+            <origin xyz="${xyz}" rpy="0 0 0"/>
+            <geometry name="${name}">
+              <box size="${size_x} ${size_y} ${size_z}"/>
+            </geometry>
+        </visual>
+        <collision>
+            <origin xyz="${xyz}" rpy="0 0 0"/>
+            <geometry>
+                <box size="${size_x} ${size_y} ${size_z}"/>
+            </geometry>
+        </collision>
+        <inertial>
+            <!-- center of mass -->
+            <origin xyz="${xyz}" rpy="0 0 0"/>
+            <mass value="${mass}"/>
+            <!-- box inertia: 1/12*m(y^2+z^2), ... -->
+            <inertia ixx="${1/12*mass*(size_y**2 + size_z**2)}" ixy="0" ixz="0"
+                iyy="${1/12*mass*(size_x**2 + size_z**2)}" iyz="0"
+                izz="${1/12*mass*(size_x**2 + size_y**2)}"/>
+          </inertial>
+    </xacro:macro>
 </robot>

File: omni_description/urdf/omnigrasper_arm/arm.xacro (robot description, xacro)
@@ -36,24 +36,27 @@
         </joint>
         <link name="arm_1">
-            <xacro:property name="arm_1_mass" value="0.855" />
+            <!-- TODO Parts to add : frame adaptor FRP54-A110K, idler FRP54-I110 -->
+            <xacro:box_vci name="arm_1" mass="0.855"
+                size_x="0.054" size_y="0.132" size_z="0.054"
+                xyz="0 0 0"/>
+            <!-- <xacro:property name="arm_1_mass" value="0.855" />
             <xacro:property name="arm_1_lx" value="0.054" />
             <xacro:property name="arm_1_ly" value="0.132" />
             <xacro:property name="arm_1_lz" value="0.054" />
-            <!-- TODO Parts to add : frame adaptor FRP54-A110K, idler FRP54-I110 -->
-            <!-- <xacro:visuals_collisions_arm_1/> -->
-            <visual> <!-- H54-200-S500 -->
+            <!-- <xacro:visuals_collisions_arm_1/> --
+            <visual> <!-- H54-200-S500 --
                 <geometry>
                     <box size="${arm_1_lx} ${arm_1_ly} ${arm_1_lz}"/>
                 </geometry>
             </visual>
-            <inertial> <!-- H54-200-S500 -->
-                <!-- center of mass -->
-                <origin rpy="0 0 0" xyz="0 0 ${0.001*(6+54/2)}"/>
+            <inertial> <!-- H54-200-S500 --
+                <!-- center of mass --
+                <origin rpy="0 0 0" xyz="0 0 0"/>
                 <mass value="${arm_1_mass}"/>
-                <!-- box inertia: 1/12*m(y^2+z^2), ... -->
+                <!-- box inertia: 1/12*m(y^2+z^2), ... --
                 <inertia ixx="${1/12*arm_1_mass*(arm_1_ly**2 + arm_1_lz**2)}" ixy="0" ixz="0"
                     iyy="${1/12*arm_1_mass*(arm_1_lx**2 + arm_1_lz**2)}" iyz="0"
                     izz="${1/12*arm_1_mass*(arm_1_lx**2 + arm_1_ly**2)}"/>
-            </inertial>
+            </inertial> -->
         </link>
         <joint name="arm_1_2" type="revolute">
@@ -70,43 +73,49 @@
             (by us) frame adaptor FRP54-H120K (modified by us), idler FRP54-I110 -->
             <!-- <xacro:visuals_collisions_arm_2/> -->
-            <xacro:property name="profile_2_mass" value="${1.38*0.180}" />
+            <xacro:box_vci name="profile_2" mass="${1.38*0.180}"
+                size_x="0.180" size_y="0.040" size_z="0.040"
+                xyz="${0.001*(51+180/2)} 0 0"/>
+            <!-- <xacro:property name="profile_2_mass" value="${1.38*0.180}" />
             <xacro:property name="profile_2_lx" value="0.180" />
             <xacro:property name="profile_2_ly" value="0.040" />
             <xacro:property name="profile_2_lz" value="0.040" />
-            <visual> <!-- aluminium profile -->
-                <origin rpy="0 0 0" xyz="${0.001*(51+180/2)} 0 0"/>
+            <visual> <!-- aluminium profile --> -->
+                <!-- <origin rpy="0 0 0" xyz="${0.001*(51+180/2)} 0 0"/>
                 <geometry name="profile_2">
                     <box size="${profile_2_lx} ${profile_2_ly} ${profile_2_lz}"/>
                 </geometry>
             </visual>
-            <inertial> <!-- aluminium profile -->
+            <inertial> <!-- aluminium profile --> -->
                 <!-- TODO: take the moments of inertia provided by manufacturer -->
                 <!-- center of mass -->
-                <origin rpy="0 0 0" xyz="${0.001*(51+180/2)} 0 0"/>
-                <mass value="${profile_2_mass}"/>
-                <!-- box inertia: 1/12*m(y^2+z^2), ... -->
-                <inertia ixx="${1/12*profile_2_mass*(profile_2_ly**2 + profile_2_lz**2)}" ixy="0" ixz="0"
+                <!-- <origin rpy="0 0 0" xyz="${0.001*(51+180/2)} 0 0"/>
+                <mass value="${profile_2_mass}"/> -->
+                <!-- box inertia: 1/12*m(y^2+z^2), ... -->
+                <!-- <inertia ixx="${1/12*profile_2_mass*(profile_2_ly**2 + profile_2_lz**2)}" ixy="0" ixz="0"
                     iyy="${1/12*profile_2_mass*(profile_2_lx**2 + profile_2_lz**2)}" iyz="0"
                     izz="${1/12*profile_2_mass*(profile_2_lx**2 + profile_2_ly**2)}"/>
-            </inertial>
-            <xacro:property name="L54_50_S500_mass" value="0.662" />
+            </inertial> -->
+            <xacro:box_vci name="L54_50_S500" mass="0.662"
+                size_x="0.054" size_y="0.054" size_z="0.114"
+                xyz="${0.001*(51+180/2)} 0 0"/>
+            <!-- <xacro:property name="L54_50_S500_mass" value="0.662" />
             <xacro:property name="L54_50_S500_lx" value="0.054" />
             <xacro:property name="L54_50_S500_ly" value="0.054" />
             <xacro:property name="L54_50_S500_lz" value="0.114" />
-            <visual> <!-- L54-50-S500 -->
-                <origin rpy="0 0 0" xyz="${0.001*(51+180+6+54/2)} 0 0"/>
-                <geometry name="L54_50_S500"> <!-- L54-50-S500 -->
-                    <box size="${L54_50_S500_lx} ${L54_50_S500_ly} ${L54_50_S500_lz}"/>
-                </geometry>
-            </visual>
-            <inertial> <!-- L54-50-S500 -->
-                <!-- center of mass -->
-                <origin rpy="0 0 0" xyz="${0.001*(51+180+6+54/2)} 0 0"/>
-                <mass value="${L54_50_S500_mass}"/>
-                <!-- box inertia: 1/12*m(y^2+z^2), ... -->
-                <inertia ixx="${1/12*L54_50_S500_mass*(L54_50_S500_ly**2 + L54_50_S500_lz**2)}" ixy="0" ixz="0"
+            <visual> <!-- L54-50-S500 --> -->
+                <!-- <origin rpy="0 0 0" xyz="${0.001*(51+180+6+54/2)} 0 0"/>
+                <geometry name="L54_50_S500"> <!-- L54-50-S500 --> -->
+                    <!-- <box size="${L54_50_S500_lx} ${L54_50_S500_ly} ${L54_50_S500_lz}"/>
+                </geometry>
+            </visual>
+            <inertial> <!-- L54-50-S500 --> -->
+                <!-- center of mass -->
+                <!-- <origin rpy="0 0 0" xyz="${0.001*(51+180+6+54/2)} 0 0"/>
+                <mass value="${L54_50_S500_mass}"/> -->
+                <!-- box inertia: 1/12*m(y^2+z^2), ... -->
+                <!-- <inertia ixx="${1/12*L54_50_S500_mass*(L54_50_S500_ly**2 + L54_50_S500_lz**2)}" ixy="0" ixz="0"
                     iyy="${1/12*L54_50_S500_mass*(L54_50_S500_lx**2 + L54_50_S500_lz**2)}" iyz="0"
                     izz="${1/12*L54_50_S500_mass*(L54_50_S500_lx**2 + L54_50_S500_ly**2)}"/>
-            </inertial>
+            </inertial> -->
         </link>
         <joint name="arm_0_1" type="revolute">

Commit message: adding colors

File: omni_description/urdf/common.xacro (robot description, xacro)
@@ -26,5 +26,5 @@
           </link>
     </xacro:macro>
-    <xacro:macro name="box_vci" params="name mass size_x size_y size_z xyz">
+    <xacro:macro name="box_vci" params="name mass size_x size_y size_z xyz color">
         <!-- For Box Visual Collision Intertial -->
         <visual>
@@ -33,4 +33,5 @@
               <box size="${size_x} ${size_y} ${size_z}"/>
             </geometry>
+            <material name="${color}"/>
         </visual>
         <collision>

File: omni_description/urdf/omnigrasper_arm/arm.urdf.xacro (robot description, xacro)
@@ -21,4 +21,5 @@
                     <box size="0.054 0.054 0.108"/>
                 </geometry>
+                <material name="omni/Blue"/>
             </visual>
         </link>
@@ -36,5 +37,5 @@
             <xacro:box_vci name="H54-200-S500" mass="0.855"
                 size_x="0.054" size_y="0.132" size_z="0.054"
-                xyz="0 0 0"/>
+                xyz="0 0 0" color="omni/Red"/>
         </link>
         <joint name="arm_1_2" type="revolute">
@@ -54,8 +55,8 @@
             <xacro:box_vci name="profile_2" mass="${1.38*0.180}"
                 size_x="0.180" size_y="0.040" size_z="0.040"
-                xyz="${0.001*(51+180/2)} 0 0"/>
+                xyz="${0.001*(51+180/2)} 0 0" color="omni/Green"/>
             <xacro:box_vci name="L54_50_S500" mass="0.662"
                 size_x="0.054" size_y="0.054" size_z="0.114"
-                xyz="${0.001*(51+180+6+54/2)} 0 0"/>
+                xyz="${0.001*(51+180+6+54/2)} 0 0" color="omni/Green"/>
         </link>
         <joint name="arm_2_3" type="revolute">
@@ -75,8 +76,8 @@
             <xacro:box_vci name="profile_3" mass="${1.38*0.060}"
                 size_x="0.040" size_y="0.060" size_z="0.040"
-                xyz="0 ${0.001*(51+60/2)} 0"/>
+                xyz="0 ${0.001*(51+60/2)} 0" color="omni/Yellow"/>
             <xacro:box_vci name="L54_30_S500" mass="0.612"
                 size_x="0.054" size_y="0.108" size_z="0.054"
-                xyz="0 ${0.001*(51+60+6+108/2)} 0"/>
+                xyz="0 ${0.001*(51+60+6+108/2)} 0" color="omni/Yellow"/>
         </link>
         <joint name="arm_3_4" type="revolute">
@@ -94,5 +95,5 @@
             <xacro:box_vci name="L42_10_S300" mass="0.257"
                 size_x="0.042" size_y="0.072" size_z="0.042"
-                xyz="0 0 0"/>
+                xyz="0 0 0" color="omni/DarkGrey"/>
         </link>
         <joint name="arm_4_5" type="revolute">
@@ -110,5 +111,5 @@
             <xacro:box_vci name="L42_10_S300" mass="0.0857"
                 size_x="0.042" size_y="0.006" size_z="0.082"
-                xyz="0 0.039 -0.006"/>
+                xyz="0 0.039 -0.006" color="omni/Blue"/>
         </link>
         <joint name="arm_5_end" type="fixed">

Commit message: adding STL files to the visual URDF

File: omni_description/urdf/common.xacro (robot description, xacro)
@@ -51,3 +51,22 @@
           </inertial>
     </xacro:macro>
+    <xacro:macro name="box_ci" params="name mass size_x size_y size_z
+        xyz color">
+        <!-- For Box Collision Intertial -->
+        <collision>
+            <origin xyz="${xyz}" rpy="0 0 0"/>
+            <geometry>
+                <box size="${size_x} ${size_y} ${size_z}"/>
+            </geometry>
+        </collision>
+        <inertial>
+            <!-- center of mass -->
+            <origin xyz="${xyz}" rpy="0 0 0"/>
+            <mass value="${mass}"/>
+            <!-- box inertia: 1/12*m(y^2+z^2), ... -->
+            <inertia ixx="${1/12*mass*(size_y**2 + size_z**2)}" ixy="0" ixz="0"
+                iyy="${1/12*mass*(size_x**2 + size_z**2)}" iyz="0"
+                izz="${1/12*mass*(size_x**2 + size_y**2)}"/>
+          </inertial>
+    </xacro:macro>
 </robot>

File: omni_description/urdf/omnigrasper_arm/arm.urdf.xacro (robot description, xacro)
@@ -16,7 +16,7 @@
         <link name="arm_0">
             <visual>
-                <origin xyz="0 0 ${-0.001*(54/2+6+108/2)}" rpy="0 0 0"/>
+                <origin xyz="0 0 ${-0.001*(54/2+6+108)}" rpy="${M_PI/2} 0 0"/>
                 <geometry>
-                    <box size="0.054 0.054 0.108"/>
+                    <mesh filename="package://omni_description/stl/L54-30-S500-R.STL" scale="0.001 0.001 0.001"/>
                 </geometry>
                 <material name="omni/Blue"/>
@@ -39,7 +39,14 @@
         <link name="arm_1">
             <!-- TODO Parts to add : frame adaptor FRP54-A110K, idler FRP54-I110 -->
-            <xacro:box_vci name="H54-200-S500" mass="0.855"
+            <xacro:box_ci name="H54-200-S500" mass="0.855"
                 size_x="0.054" size_y="0.132" size_z="0.054"
                 xyz="0 0 0" color="omni/Red"/>
+            <visual>
+                <origin xyz="0 ${-0.132/2} 0"/>
+                <geometry>
+                    <mesh filename="package://omni_description/stl/H54-200-S500-R.STL" scale="0.001 0.001 0.001"/>
+                </geometry>
+                <material name="omni/Red"/>
+            </visual>
         </link>
         <joint name="arm_1_2" type="revolute">
@@ -65,7 +72,15 @@
         </joint>
         <link name="arm_2_sub">
-            <xacro:box_vci name="L54_50_S500" mass="0.662"
+            <xacro:box_ci name="L54_50_S500" mass="0.662"
                 size_x="0.054" size_y="0.054" size_z="0.114"
                 xyz="${0.001*(51+180+6+54/2)} 0 0" color="omni/Green"/>
+            <visual>
+                <origin xyz="${0.001*(51+180+6+54/2)} 0 ${0.114/2}"
+                    rpy="${-M_PI/2} 0 0"/>
+                <geometry>
+                    <mesh filename="package://omni_description/stl/L54-50-S500-R.STL" scale="0.001 0.001 0.001"/>
+                </geometry>
+                <material name="omni/Green"/>
+            </visual>
         </link>
         <joint name="arm_2_3" type="revolute">
@@ -91,7 +106,14 @@
         </joint>
         <link name="arm_3_sub">
-            <xacro:box_vci name="L54_30_S500" mass="0.612"
+            <xacro:box_ci name="L54_30_S500" mass="0.612"
                 size_x="0.054" size_y="0.108" size_z="0.054"
                 xyz="0 ${0.001*(51+60+6+108/2)} 0" color="omni/Yellow"/>
+            <visual>
+                <origin xyz="0 ${0.001*(51+60+6)} 0" rpy="0 ${-M_PI} 0"/>
+                <geometry>
+                    <mesh filename="package://omni_description/stl/L54-30-S500-R.STL" scale="0.001 0.001 0.001"/>
+                </geometry>
+                <material name="omni/Yellow"/>
+            </visual>
         </link>
         <joint name="arm_3_4" type="revolute">
@@ -105,7 +127,14 @@
             <!-- TODO Parts to add : modified (by us) frame adaptor FRP54-A110K,
             idler FRP42-I110 -->
-            <xacro:box_vci name="L42_10_S300" mass="0.257"
+            <xacro:box_ci name="L42_10_S300" mass="0.257"
                 size_x="0.042" size_y="0.072" size_z="0.042"
                 xyz="0 0 0" color="omni/DarkGrey"/>
+            <visual>
+                <origin xyz="0 ${-0.072/2} 0" rpy="0 0 0"/>
+                <geometry>
+                    <mesh filename="package://omni_description/stl/L42-10-S300-R.STL" scale="0.001 0.001 0.001"/>
+                </geometry>
+                <material name="omni/DarkGrey"/>
+            </visual>
         </link>
         <joint name="arm_4_5" type="revolute">
